File: eagle/thrust_stand.brd (EAGLE design)
At the start: 100 x 80 mm, 27 parts, among them IC1 7805TV, Q1 16Mhz, Q2 IRF510, T1 2N3904, U2 ATMEGA328P_PDIP

Commit message: tweaks
Parts:
- moved R1 9.16 mm to (26.7, 36.8), turned to 270 degrees
- moved HX711 8.13 mm to (17.8, 25.4)
- moved IGN1 7.62 mm to (59.7, 16.5)
- moved I2C_2 6.35 mm to (7.62, 26.7)
- moved I2C_3 6.35 mm to (7.62, 20.3)
- moved I2C_1 6.35 mm to (7.62, 33.0)
- moved RESET 5.39 mm to (21.6, 36.8)
- moved Q2 5.24 mm to (53.3, 10.2), turned to 0 degrees
- moved R5 4.02 mm to (49.5, 16.5)
- moved R2 3.59 mm to (53.3, 16.5)
- moved BATTERY 2.84 mm to (49.5, 38.1)
- turned LED1 to 0 degrees
